Commit message: Add files via upload

File: urdf/wally.xacro (robot description, xacro)
@@ -5,6 +5,6 @@
   <link name="base_link">
     <inertial>
-      <origin xyz="-0.0083636 0.0065553 0.033694" rpy="0 0 0" />
-      <mass value="1.4521" />
+      <origin xyz="0 0 0" rpy="0 0 0" />
+      <mass value="1.5" />
       <inertia ixx="0.0040255" ixy="-2.6373E-06" ixz="6.2085E-08" iyy="0.0046487" iyz="-1.1645E-06" izz="0.0086266" />
     </inertial>

Commit message: Add files via upload

File: urdf/wally.xacro (robot description, xacro)
@@ -2,163 +2,94 @@
 <robot name="wally" xmlns:xacro="http://www.ros.org/wiki/xacro">
   <xacro:include filename="$(find wally_description)/urdf/wally.gazebo" />
-  <xacro:include filename="$(find wally_description)/urdf/materials.xacro" />
   <link name="base_link">
     <inertial>
       <origin xyz="0 0 0" rpy="0 0 0" />
-      <mass value="1.5" />
-      <inertia ixx="0.0040255" ixy="-2.6373E-06" ixz="6.2085E-08" iyy="0.0046487" iyz="-1.1645E-06" izz="0.0086266" />
-    </inertial>
-    <visual>
-      <origin xyz="0 0 0" rpy="0 0 0" />
-      <geometry>
-	<mesh filename="package://wally_description/meshes/base_link.STL" />
-      </geometry>
-      <material name="base">
-	<color rgba="0.8 0.8 0.8 1" />
-      </material>
-    </visual>
-    <collision>
-      <origin xyz="0 0 0" rpy="0 0 0" />
-      <geometry>
-	<mesh filename="package://wally_description/meshes/base_link.STL" />
-      </geometry>
-    </collision>
-  </link>
-  <link name="motor_A">
-    <inertial>
-      <origin xyz="-4.1573E-07 -6.9339E-08 0.0137" rpy="0 0 0" />
-      <mass value="0.047845" />
-      <inertia ixx="1.9654E-05" ixy="9.7041E-10" ixz="-1.1174E-11" iyy="1.9654E-05" iyz="1.3746E-10" izz="3.4083E-05" />
-    </inertial>
-    <visual>
-      <origin xyz="0 0 0" rpy="0 0 0" />
-      <geometry>
-	<mesh filename="package://wally_description/meshes/motor_A.STL" />
-      </geometry>
-      <material name="motorA">
-	<color rgba="0.77647 0.55686 0.10588 1" />
-      </material>
-    </visual>
-    <collision>
-      <origin xyz="0 0 0" rpy="0 0 0" />
-      <geometry>
-	<mesh filename="package://wally_description/meshes/motor_A.STL" />
-      </geometry>
-    </collision>
-  </link>
-  <joint name="joint_A" type="continuous">
-    <origin xyz="-0.1269 -0.11168 -0.021875" rpy="-1.5708 0.51523 1.5708" />
-    <parent link="base_link" />
-    <child link="motor_A" />
-    <axis xyz="0 0 -1" />
-  </joint>
-  <link name="motor_B">
-    <inertial>
-      <origin xyz="-4.1576E-07 -6.9176E-08 0.0137" rpy="0 0 0" />
-      <mass value="0.047845" />
-      <inertia ixx="1.9654E-05" ixy="9.7024E-10" ixz="-1.128E-11" iyy="1.9654E-05" iyz="1.3737E-10" izz="3.4083E-05" />
-    </inertial>
-    <visual>
-      <origin xyz="0 0 0" rpy="0 0 0" />
-      <geometry>
-	<mesh filename="package://wally_description/meshes/motor_B.STL" />
-      </geometry>
-      <material name="motorB">
-	<color rgba="0.77647 0.55686 0.10588 1" />
-      </material>
-    </visual>
-    <collision>
-      <origin xyz="0 0 0" rpy="0 0 0" />
-      <geometry>
-	<mesh filename="package://wally_description/meshes/motor_B.STL" />
-      </geometry>
-    </collision>
-  </link>
-  <joint name="joint_B" type="continuous">
-    <origin xyz="0.1269 -0.11168 -0.021875" rpy="-1.5708 -0.57038 -1.5708" />
-    <parent link="base_link" />
-    <child link="motor_B" />
-    <axis xyz="0 0 1" />
-  </joint>
-  <link name="motor_C">
-    <inertial>
-      <origin xyz="4.1469E-07 6.8439E-08 0.0137" rpy="0 0 0" />
-      <mass value="0.047845" />
-      <inertia ixx="1.9654E-05" ixy="9.7024E-10" ixz="1.0734E-11" iyy="1.9654E-05" iyz="-1.38E-10" izz="3.4083E-05" />
-    </inertial>
-    <visual>
-      <origin xyz="0 0 0" rpy="0 0 0" />
-      <geometry>
-	<mesh filename="package://wally_description/meshes/motor_C.STL" />
-      </geometry>
-      <material name="motorC">
-	<color rgba="0.77647 0.55686 0.10588 1" />
-      </material>
-    </visual>
-    <collision>
-      <origin xyz="0 0 0" rpy="0 0 0" />
-      <geometry>
-	<mesh filename="package://wally_description/meshes/motor_C.STL" />
-      </geometry>
-    </collision>
-  </link>
-  <joint name="joint_C" type="continuous">
-    <origin xyz="0.1269 0.11168 -0.021875" rpy="1.5708 -0.50447 1.5708" />
-    <parent link="base_link" />
-    <child link="motor_C" />
-    <axis xyz="0 0 1" />
-  </joint>
-  <link name="motor_D">
-    <inertial>
-      <origin xyz="4.1418E-07 6.8329E-08 0.0137" rpy="0 0 0" />
-      <mass value="0.047845" />
-      <inertia ixx="1.9654E-05" ixy="9.7033E-10" ixz="1.0826E-11" iyy="1.9654E-05" iyz="-1.3801E-10" izz="3.4083E-05" />
-    </inertial>
-    <visual>
-      <origin xyz="0 0 0" rpy="0 0 0" />
-      <geometry>
-	<mesh filename="package://wally_description/meshes/motor_D.STL" />
-      </geometry>
-      <material name="motorD">
-	<color rgba="0.77647 0.55686 0.10588 1" />
-      </material>
-    </visual>
-    <collision>
-      <origin xyz="0 0 0" rpy="0 0 0" />
-      <geometry>
-	<mesh filename="package://wally_description/meshes/motor_D.STL" />
-      </geometry>
-    </collision>
-  </link>
-  <joint name="joint_D" type="continuous">
-    <origin xyz="-0.1269 0.11168 -0.021875" rpy="1.5708 -0.62108 -1.5708" />
-    <parent link="base_link" />
-    <child link="motor_D" />
-    <axis xyz="0 0 -1" />
+      <mass value="0.380" />
+      <inertia ixx="0.004708822" ixy="9.04E-07" ixz="0" iyy="0.004514873" iyz="0" izz="0.009096925" />
+    </inertial>
+    <visual>
+      <origin xyz="0 0 0" rpy="0 0 1.57075" />
+      <geometry>
+	<mesh filename="package://wally_description/meshes/BASE01.dae" />
+      </geometry>
+    </visual>
+    <collision>
+      <origin xyz="0 0 0" rpy="0 0 1.57075" />
+      <geometry>
+	<mesh filename="package://wally_description/meshes/BASE01.dae" />
+      </geometry>
+    </collision>
+  </link>
+  <link name="Base_02">
+    <inertial>
+      <origin xyz="0 0 0.06" rpy="0 0 0" />
+      <mass value="0.380" />
+      <inertia ixx="0.004708822" ixy="9.04E-07" ixz="0" iyy="0.004514873" iyz="0" izz="0.009096925" />
+    </inertial>
+    <visual>
+      <origin xyz="0 0 0.06" rpy="0 0 0" />
+      <geometry>
+	<mesh filename="package://wally_description/meshes/BASE02.dae" />
+      </geometry>
+    </visual>
+    <collision>
+      <origin xyz="0 0 0.06" rpy="0 0 0" />
+      <geometry>
+	<mesh filename="package://wally_description/meshes/BASE02.dae" />
+      </geometry>
+    </collision>
+  </link>
+  <joint name="base02" type="fixed">
+    <origin xyz="0 0 0" rpy="0 0 1.57075" />
+    <parent link="base_link" />
+    <child link="Base_02" />
+    <axis xyz="0 0 0" />
+  </joint>
+  <link name="Base_03">
+    <inertial>
+      <origin xyz="0 0 0.119" rpy="0 0 0" />
+      <mass value="0.095" />
+      <inertia ixx="0.000085867" ixy="0" ixz="0" iyy="0.000532995" iyz="0" izz="0.00061183" />
+    </inertial>
+    <visual>
+      <origin xyz="0 0 0.119" rpy="0 0 0" />
+      <geometry>
+	<mesh filename="package://wally_description/meshes/BASE03.dae" />
+      </geometry>
+    </visual>
+    <collision>
+      <origin xyz="0 0 0.119" rpy="0 0 0" />
+      <geometry>
+	<mesh filename="package://wally_description/meshes/BASE03.dae" />
+      </geometry>
+    </collision>
+  </link>
+  <joint name="base03" type="fixed">
+    <origin xyz="0 0 0" rpy="0 0 1.57075" />
+    <parent link="base_link" />
+    <child link="Base_03" />
+    <axis xyz="0 0 0" />
   </joint>
   <link name="ZED">
     <inertial>
-      <origin xyz="2.2764E-08 -2.8942E-06 0.015659" rpy="0 0 0" />
-      <mass value="0.14788" />
-      <inertia ixx="2.1445E-05" ixy="2.4719E-11" ixz="-1.7198E-11" iyy="0.00036611" iyz="-7.0654E-09" izz="0.00036349" />
-    </inertial>
-    <visual>
-      <origin xyz="0 0 0" rpy="0 0 0" />
-      <geometry>
-	<mesh filename="package://wally_description/meshes/ZED.STL" />
-      </geometry>
-      <material name="">
-	<color rgba="0.89804 0.91373 0.92549 1" />
-      </material>
-    </visual>
-    <collision>
-      <origin xyz="0 0 0" rpy="0 0 0" />
-      <geometry>
-	<mesh filename="package://wally_description/meshes/ZED.STL" />
+      <origin xyz="0 -0.08935 0.076485" rpy="0 0 0" />
+      <mass value="0.135" />
+      <inertia ixx="0.000021510" ixy="0" ixz="0" iyy="0.000366159" iyz="0" izz="0.000363493" />
+    </inertial>
+    <visual>
+      <origin xyz="0 -0.08935 0.076485" rpy="0 0 0" />
+      <geometry>
+	<mesh filename="package://wally_description/meshes/ZED.dae" />
+      </geometry>
+    </visual>
+    <collision>
+      <origin xyz="0 -0.08935 0.076485" rpy="0 0 0" />
+      <geometry>
+	<mesh filename="package://wally_description/meshes/ZED.dae" />
       </geometry>
     </collision>
   </link>
   <joint name="camera" type="fixed">
-    <origin xyz="0 -0.0736 0.076488" rpy="1.5708 0 0" />
+    <origin xyz="0 0 0" rpy="0 0 1.57075" />
     <parent link="base_link" />
     <child link="ZED" />
@@ -167,28 +98,125 @@
   <link name="RP_LIDAR">
     <inertial>
-      <origin xyz="0 0 0" rpy="0 0 0" />
-      <mass value="1e-5" />
-      <inertia ixx="1e-6" ixy="0" ixz="0" iyy="1e-6" iyz="0" izz="1e-6" />
-    </inertial>
-    <visual>
-      <origin xyz="0 0 -0.037" rpy="1.5708 0 3.14159" />
-      <geometry>
-	<mesh filename="package://wally_description/meshes/rp_lidarA1.stl" scale="0.01 0.01 0.01"/>
-      </geometry>
-      <material name="lidar">
-	<color rgba="0.75294 0.75294 0.75294 1" />
-      </material>
-    </visual>
-    <collision>
-      <origin xyz="0 0 0" rpy="0 0 0" />
-      <geometry>
-	<mesh filename="package://wally_description/meshes/rp_lidarA1.stl" scale="0.01 0.01 0.01"/>
+      <origin xyz="0 0 0.1205" rpy="0 0 0" />
+      <mass value="0.170" />
+      <inertia ixx="0.000117046" ixy="-2.01E-07" ixz="-4.01E-07" iyy="0.000076301" iyz="0.000014883" izz="0.000082665" />
+    </inertial>
+    <visual>
+      <origin xyz="0 0 0.1205" rpy="0 0 0" />
+      <geometry>
+	<mesh filename="package://wally_description/meshes/RP_LIDAR.dae" />
+      </geometry>
+    </visual>
+    <collision>
+      <origin xyz="0 0 0.1205" rpy="0 0 0" />
+      <geometry>
+	<mesh filename="package://wally_description/meshes/RP_LIDAR.dae" />
       </geometry>
     </collision>
   </link>
   <joint name="lidar" type="fixed">
-    <origin xyz="0 0 0.158" rpy="0 0 -1.5708" />
+    <origin xyz="0 0 0" rpy="0 0 1.57075" />
     <parent link="base_link" />
     <child link="RP_LIDAR" />
+    <axis xyz="0 0 1" />
+  </joint>
+  <link name="motor_A">
+    <inertial>
+      <origin xyz="-0.11168 0 0.021875" rpy="0 0 3.1415" />
+      <mass value="0.061" />
+      <inertia ixx="0.000034341" ixy="0" ixz="0" iyy="0.000020393" iyz="0" izz="0.000020401" />
+    </inertial>
+    <visual>
+      <origin xyz="-0.11168 0 0.021875" rpy="0 0 3.1415" />
+      <geometry>
+	<mesh filename="package://wally_description/meshes/RODA_A.dae" />
+      </geometry>
+    </visual>
+    <collision>
+      <origin xyz="-0.11168 0 0.021875" rpy="0 0 3.1415" />
+      <geometry>
+	<mesh filename="package://wally_description/meshes/RODA_A.dae" />
+      </geometry>
+    </collision>
+  </link>
+  <joint name="joint_A" type="continuous">
+    <origin xyz="0.111681 0 -0.021875" rpy="0 0 0"/>
+    <parent link="base_link" />
+    <child link="motor_A" />
+    <axis xyz="0 1 0" />
+  </joint>
+  <link name="motor_B">
+    <inertial>
+      <origin xyz="-0.11168 0 -0.021875" rpy="3.1415 0 3.1415" />
+      <mass value="0.061" />
+      <inertia ixx="0.000034341" ixy="0" ixz="0" iyy="0.000020393" iyz="0" izz="0.000020401" />
+    </inertial>
+    <visual>
+      <origin xyz="-0.11168 0 -0.021875" rpy="3.1415 0 3.1415" />
+      <geometry>
+	<mesh filename="package://wally_description/meshes/RODA_A.dae" />
+      </geometry>
+    </visual>
+    <collision>
+      <origin xyz="-0.11168 0 -0.021875" rpy="3.1415 0 3.1415" />
+      <geometry>
+	<mesh filename="package://wally_description/meshes/RODA_A.dae" />
+      </geometry>
+    </collision>
+  </link>
+  <joint name="joint_B" type="continuous">
+    <origin xyz="0.11168 0 -0.021875" rpy="0 3.1415 0" />
+    <parent link="base_link" />
+    <child link="motor_B" />
+    <axis xyz="0 1 0" />
+  </joint>
+  <link name="motor_C">
+    <inertial>
+      <origin xyz="0.11168 0 0.021875" rpy="0 0 0" />
+      <mass value="0.061" />
+      <inertia ixx="0.000034341" ixy="0" ixz="0" iyy="0.000020393" iyz="0" izz="0.000020401" />
+    </inertial>
+    <visual>
+      <origin xyz="0.11168 0 0.021875" rpy="0 0 0" />
+      <geometry>
+	<mesh filename="package://wally_description/meshes/RODA_A.dae" />
+      </geometry>
+    </visual>
+    <collision>
+      <origin xyz="0.11168 0 0.021875" rpy="0 0 0" />
+      <geometry>
+	<mesh filename="package://wally_description/meshes/RODA_A.dae" />
+      </geometry>
+    </collision>
+  </link>
+  <joint name="joint_C" type="continuous">
+    <origin xyz="-0.11168 0 -0.021875" rpy="0 0 0" />
+    <parent link="base_link" />
+    <child link="motor_C" />
+    <axis xyz="0 1 0" />
+  </joint>
+  <link name="motor_D">
+    <inertial>
+      <origin xyz="0.11168 0 -0.021875" rpy="3.1415 0 0" />
+      <mass value="0.061" />
+      <inertia ixx="0.000034341" ixy="0" ixz="0" iyy="0.000020393" iyz="0" izz="0.000020401" />
+    </inertial>
+    <visual>
+      <origin xyz="0.11168 0 -0.021875" rpy="3.1415 0 0" />
+      <geometry>
+	<mesh filename="package://wally_description/meshes/RODA_A.dae" />
+      </geometry>
+    </visual>
+    <collision>
+      <origin xyz="0.11168 0 -0.021875" rpy="3.1415 0 0" />
+      <geometry>
+	<mesh filename="package://wally_description/meshes/RODA_A.dae" />
+      </geometry>
+    </collision>
+  </link>
+  <joint name="joint_D" type="continuous">
+    <origin xyz="-0.11168 0 -0.021875" rpy="0 0 0" />
+    <parent link="base_link" />
+    <child link="motor_D" />
     <axis xyz="0 1 0" />
   </joint>

Commit message: Add files via upload

File: urdf/wally.xacro (robot description, xacro)
@@ -5,6 +5,6 @@
     <inertial>
       <origin xyz="0 0 0" rpy="0 0 0" />
-      <mass value="0.380" />
-      <inertia ixx="0.004708822" ixy="9.04E-07" ixz="0" iyy="0.004514873" iyz="0" izz="0.009096925" />
+      <mass value="4.380" />
+      <inertia ixx="0.000003" ixy="0" ixz="0" iyy="0.000003" iyz="0" izz="0.000005" />
     </inertial>
     <visual>
@@ -25,5 +25,5 @@
       <origin xyz="0 0 0.06" rpy="0 0 0" />
       <mass value="0.380" />
-      <inertia ixx="0.004708822" ixy="9.04E-07" ixz="0" iyy="0.004514873" iyz="0" izz="0.009096925" />
+      <inertia ixx="0.000002" ixy="0" ixz="0" iyy="0.000002" iyz="0" izz="0.000003" />
     </inertial>
     <visual>
@@ -50,5 +50,5 @@
       <origin xyz="0 0 0.119" rpy="0 0 0" />
       <mass value="0.095" />
-      <inertia ixx="0.000085867" ixy="0" ixz="0" iyy="0.000532995" iyz="0" izz="0.00061183" />
+      <inertia ixx="0" ixy="0" ixz="0" iyy="0" iyz="0" izz="0" />
     </inertial>
     <visual>
@@ -75,5 +75,5 @@
       <origin xyz="0 -0.08935 0.076485" rpy="0 0 0" />
       <mass value="0.135" />
-      <inertia ixx="0.000021510" ixy="0" ixz="0" iyy="0.000366159" iyz="0" izz="0.000363493" />
+      <inertia ixx="0" ixy="0" ixz="0" iyy="0" iyz="0" izz="0" />
     </inertial>
     <visual>
@@ -100,21 +100,21 @@
       <origin xyz="0 0 0.1205" rpy="0 0 0" />
       <mass value="0.170" />
-      <inertia ixx="0.000117046" ixy="-2.01E-07" ixz="-4.01E-07" iyy="0.000076301" iyz="0.000014883" izz="0.000082665" />
-    </inertial>
-    <visual>
+      <inertia ixx="0.000117046" ixy="0" ixz="0" iyy="0.000076301" iyz="0" izz="0.000082665" />
+    </inertial>
+    <visual>
+      <origin xyz="0 0 -0.045" rpy="0 0 0" />
+      <geometry>
+	<mesh filename="package://wally_description/meshes/RP_LIDAR.dae" />
+      </geometry>
+    </visual>
+    <collision>
       <origin xyz="0 0 0.1205" rpy="0 0 0" />
       <geometry>
 	<mesh filename="package://wally_description/meshes/RP_LIDAR.dae" />
       </geometry>
-    </visual>
-    <collision>
-      <origin xyz="0 0 0.1205" rpy="0 0 0" />
-      <geometry>
-	<mesh filename="package://wally_description/meshes/RP_LIDAR.dae" />
-      </geometry>
     </collision>
   </link>
   <joint name="lidar" type="fixed">
-    <origin xyz="0 0 0" rpy="0 0 1.57075" />
+    <origin xyz="0 0 0.1655" rpy="0 0 1.57075" />
     <parent link="base_link" />
     <child link="RP_LIDAR" />
@@ -125,5 +125,5 @@
       <origin xyz="-0.11168 0 0.021875" rpy="0 0 3.1415" />
       <mass value="0.061" />
-      <inertia ixx="0.000034341" ixy="0" ixz="0" iyy="0.000020393" iyz="0" izz="0.000020401" />
+      <inertia ixx="0.002" ixy="0" ixz="0" iyy="0.002" iyz="0" izz="0.002" />
     </inertial>
     <visual>
@@ -150,5 +150,5 @@
       <origin xyz="-0.11168 0 -0.021875" rpy="3.1415 0 3.1415" />
       <mass value="0.061" />
-      <inertia ixx="0.000034341" ixy="0" ixz="0" iyy="0.000020393" iyz="0" izz="0.000020401" />
+      <inertia ixx="0.002" ixy="0" ixz="0" iyy="0.002" iyz="0" izz="0.002" />
     </inertial>
     <visual>
@@ -175,5 +175,5 @@
       <origin xyz="0.11168 0 0.021875" rpy="0 0 0" />
       <mass value="0.061" />
-      <inertia ixx="0.000034341" ixy="0" ixz="0" iyy="0.000020393" iyz="0" izz="0.000020401" />
+      <inertia ixx="0.002" ixy="0" ixz="0" iyy="0.002" iyz="0" izz="0.002" />
     </inertial>
     <visual>
@@ -200,5 +200,5 @@
       <origin xyz="0.11168 0 -0.021875" rpy="3.1415 0 0" />
       <mass value="0.061" />
-      <inertia ixx="0.000034341" ixy="0" ixz="0" iyy="0.000020393" iyz="0" izz="0.000020401" />
+      <inertia ixx="0.002" ixy="0" ixz="0" iyy="0.002" iyz="0" izz="0.002" />
     </inertial>
     <visual>
@@ -221,3 +221,128 @@
     <axis xyz="0 1 0" />
   </joint>
+    <link name="Arduino_Due">
+    <inertial>
+      <origin xyz="-0.0132 -0.04333 0.0053" rpy="0 0 1.57075" />
+      <mass value="0.035" />
+      <inertia ixx="0" ixy="0" ixz="0" iyy="0" iyz="0" izz="0" />
+    </inertial>
+    <visual>
+      <origin xyz="0.04333 -0.0132 0.0053" rpy="0 0 1.57075" />
+      <geometry>
+	<mesh filename="package://wally_description/meshes/ARDUINO_DUE.dae" />
+      </geometry>
+    </visual>
+    <collision>
+      <origin xyz="-0.0132 -0.04333 0.0053" rpy="0 0 1.57075" />
+      <geometry>
+	<mesh filename="package://wally_description/meshes/ARDUINO_DUE.dae" />
+      </geometry>
+    </collision>
+  </link>
+  <joint name="arduino" type="fixed">
+    <origin xyz="0 0 0" rpy="0 0 0" />
+    <parent link="base_link" />
+    <child link="Arduino_Due" />
+    <axis xyz="0 0 1" />
+  </joint>
+  <link name="Bateria">
+    <inertial>
+      <origin xyz="0 -0.108 0.0145" rpy="0 0 -1.57075" />
+      <mass value="0.45" />
+      <inertia ixx="0" ixy="0" ixz="0" iyy="0" iyz="0" izz="0" />
+    </inertial>
+    <visual>
+      <origin xyz="0 -0.108 0.0145" rpy="0 0 -1.5707" />
+      <geometry>
+	<mesh filename="package://wally_description/meshes/BATERIA.dae" />
+      </geometry>
+    </visual>
+    <collision>
+      <origin xyz="0 -0.108 0.0145" rpy="0 0 -1.57075" />
+      <geometry>
+	<mesh filename="package://wally_description/meshes/BATERIA.dae" />
+      </geometry>
+    </collision>
+  </link>
+  <joint name="bateria" type="fixed">
+    <origin xyz="0 0 0" rpy="0 0 1.57075" />
+    <parent link="base_link" />
+    <child link="Bateria" />
+    <axis xyz="0 0 1" />
+  </joint>
+  <link name="Hub_usb">
+    <inertial>
+      <origin xyz="0 0.0995 0.0115" rpy="0 0 1.57075" />
+      <mass value="0.03" />
+      <inertia ixx="0" ixy="0" ixz="0" iyy="0" iyz="0" izz="0" />
+    </inertial>
+    <visual>
+      <origin xyz="0 0.0995 0.0115" rpy="0 0 1.57075" />
+      <geometry>
+	<mesh filename="package://wally_description/meshes/HUB_USB.dae" />
+      </geometry>
+    </visual>
+    <collision>
+      <origin xyz="0 0.0995 0.0115" rpy="0 0 1.57075" />
+      <geometry>
+	<mesh filename="package://wally_description/meshes/HUB_USB.dae" />
+      </geometry>
+    </collision>
+  </link>
+  <joint name="hub" type="fixed">
+    <origin xyz="0 0 0" rpy="0 0 0" />
+    <parent link="base_link" />
+    <child link="Hub_usb" />
+    <axis xyz="0 0 1" />
+  </joint>
+  <link name="Power_bank">
+    <inertial>
+      <origin xyz="-0.028 -0.002 0.013" rpy="0 3.1415 0" />
+      <mass value="0.6" />
+      <inertia ixx="0.000001" ixy="0" ixz="0" iyy="0" iyz="0" izz="0.000001" />
+    </inertial>
+    <visual>
+      <origin xyz="-0.028 -0.002 0.013" rpy="0 3.1415 0" />
+      <geometry>
+	<mesh filename="package://wally_description/meshes/POWER_BANK.dae" />
+      </geometry>
+    </visual>
+    <collision>
+      <origin xyz="-0.028 -0.002 0.013" rpy="0 3.1415 0" />
+      <geometry>
+	<mesh filename="package://wally_description/meshes/POWER_BANK.dae" />
+      </geometry>
+    </collision>
+  </link>
+  <joint name="power_bank" type="fixed">
+    <origin xyz="0 0 0" rpy="0 0 0" />
+    <parent link="base_link" />
+    <child link="Power_bank" />
+    <axis xyz="0 0 1" />
+  </joint>
+  <link name="Jetson">
+    <inertial>
+      <origin xyz="-0.017 0 0.0625" rpy="0 0 0" />
+      <mass value="0.5" />
+      <inertia ixx="0" ixy="0" ixz="0" iyy="0" iyz="0" izz="0" />
+    </inertial>
+    <visual>
+      <origin xyz="-0.017 0 0.0625" rpy="0 0 0" />
+      <geometry>
+	<mesh filename="package://wally_description/meshes/JETSON.dae" />
+      </geometry>
+    </visual>
+    <collision>
+      <origin xyz="-0.017 0 0.0625" rpy="0 0 0" />
+      <geometry>
+	<mesh filename="package://wally_description/meshes/JETSON.dae" />
+      </geometry>
+    </collision>
+  </link>
+  <joint name="jetson" type="fixed">
+    <origin xyz="0 0 0" rpy="0 0 0" />
+    <parent link="base_link" />
+    <child link="Jetson" />
+    <axis xyz="0 0 1" />
+  </joint>
 </robot>

Commit message: Add files via upload

File: urdf/wally.xacro (robot description, xacro)
@@ -6,5 +6,5 @@
       <origin xyz="0 0 0" rpy="0 0 0" />
       <mass value="4.380" />
-      <inertia ixx="0.000003" ixy="0" ixz="0" iyy="0.000003" iyz="0" izz="0.000005" />
+      <inertia ixx="1.000003" ixy="0" ixz="0" iyy="1.000003" iyz="0" izz="1.000005" />
     </inertial>
     <visual>
