Commit message: Add files via upload

File: urdf/wally.xacro (robot description, xacro)
@@ -98,10 +98,10 @@
   <link name="RP_LIDAR">
     <inertial>
-      <origin xyz="0 0 0.1205" rpy="0 0 0" />
+      <origin xyz="0 0 0.1205" rpy="0 0 -1.57075" />
       <mass value="0.170" />
       <inertia ixx="0.000117046" ixy="0" ixz="0" iyy="0.000076301" iyz="0" izz="0.000082665" />
     </inertial>
     <visual>
-      <origin xyz="0 0 -0.045" rpy="0 0 0" />
+      <origin xyz="0 0 -0.045" rpy="0 0 -1.57075" />
       <geometry>
 	<mesh filename="package://wally_description/meshes/RP_LIDAR.dae" />
@@ -109,5 +109,5 @@
     </visual>
     <collision>
-      <origin xyz="0 0 0.1205" rpy="0 0 0" />
+      <origin xyz="0 0 0.1205" rpy="0 0 -1.57075" />
       <geometry>
 	<mesh filename="package://wally_description/meshes/RP_LIDAR.dae" />
@@ -116,5 +116,5 @@
   </link>
   <joint name="lidar" type="fixed">
-    <origin xyz="0 0 0.1655" rpy="0 0 1.57075" />
+    <origin xyz="0 0 0.1655" rpy="0 0 3.1415" />
     <parent link="base_link" />
     <child link="RP_LIDAR" />

Commit message: Update wally.xacro

File: urdf/wally.xacro (robot description, xacro)
@@ -121,5 +121,5 @@
     <axis xyz="0 0 1" />
   </joint>
-  <link name="motor_A">
+  <link name="roda_A">
     <inertial>
       <origin xyz="-0.11168 0 0.021875" rpy="0 0 3.1415" />
@@ -143,8 +143,8 @@
     <origin xyz="0.111681 0 -0.021875" rpy="0 0 0"/>
     <parent link="base_link" />
-    <child link="motor_A" />
+    <child link="roda_A" />
     <axis xyz="0 1 0" />
   </joint>
-  <link name="motor_B">
+  <link name="roda_B">
     <inertial>
       <origin xyz="-0.11168 0 -0.021875" rpy="3.1415 0 3.1415" />
@@ -168,8 +168,8 @@
     <origin xyz="0.11168 0 -0.021875" rpy="0 3.1415 0" />
     <parent link="base_link" />
-    <child link="motor_B" />
+    <child link="roda_B" />
     <axis xyz="0 1 0" />
   </joint>
-  <link name="motor_C">
+  <link name="roda_C">
     <inertial>
       <origin xyz="0.11168 0 0.021875" rpy="0 0 0" />
@@ -193,8 +193,8 @@
     <origin xyz="-0.11168 0 -0.021875" rpy="0 0 0" />
     <parent link="base_link" />
-    <child link="motor_C" />
+    <child link="roda_C" />
     <axis xyz="0 1 0" />
   </joint>
-  <link name="motor_D">
+  <link name="roda_D">
     <inertial>
       <origin xyz="0.11168 0 -0.021875" rpy="3.1415 0 0" />
@@ -218,5 +218,5 @@
     <origin xyz="-0.11168 0 -0.021875" rpy="0 0 0" />
     <parent link="base_link" />
-    <child link="motor_D" />
+    <child link="roda_D" />
     <axis xyz="0 1 0" />
   </joint>

Commit message: Add files via upload

File: urdf/wally.xacro (robot description, xacro)
@@ -130,5 +130,5 @@
       <origin xyz="-0.11168 0 0.021875" rpy="0 0 3.1415" />
       <geometry>
-	<mesh filename="package://wally_description/meshes/RODA_A.dae" />
+	<mesh filename="package://wally_description/meshes/RODA.dae" />
       </geometry>
     </visual>
@@ -136,5 +136,5 @@
       <origin xyz="-0.11168 0 0.021875" rpy="0 0 3.1415" />
       <geometry>
-	<mesh filename="package://wally_description/meshes/RODA_A.dae" />
+	<mesh filename="package://wally_description/meshes/RODA.dae" />
       </geometry>
     </collision>
@@ -155,5 +155,5 @@
       <origin xyz="-0.11168 0 -0.021875" rpy="3.1415 0 3.1415" />
       <geometry>
-	<mesh filename="package://wally_description/meshes/RODA_A.dae" />
+	<mesh filename="package://wally_description/meshes/RODA.dae" />
       </geometry>
     </visual>
@@ -161,5 +161,5 @@
       <origin xyz="-0.11168 0 -0.021875" rpy="3.1415 0 3.1415" />
       <geometry>
-	<mesh filename="package://wally_description/meshes/RODA_A.dae" />
+	<mesh filename="package://wally_description/meshes/RODA.dae" />
       </geometry>
     </collision>
@@ -180,5 +180,5 @@
       <origin xyz="0.11168 0 0.021875" rpy="0 0 0" />
       <geometry>
-	<mesh filename="package://wally_description/meshes/RODA_A.dae" />
+	<mesh filename="package://wally_description/meshes/RODA.dae" />
       </geometry>
     </visual>
@@ -186,5 +186,5 @@
       <origin xyz="0.11168 0 0.021875" rpy="0 0 0" />
       <geometry>
-	<mesh filename="package://wally_description/meshes/RODA_A.dae" />
+	<mesh filename="package://wally_description/meshes/RODA.dae" />
       </geometry>
     </collision>
@@ -205,5 +205,5 @@
       <origin xyz="0.11168 0 -0.021875" rpy="3.1415 0 0" />
       <geometry>
-	<mesh filename="package://wally_description/meshes/RODA_A.dae" />
+	<mesh filename="package://wally_description/meshes/RODA.dae" />
       </geometry>
     </visual>
@@ -211,5 +211,5 @@
       <origin xyz="0.11168 0 -0.021875" rpy="3.1415 0 0" />
       <geometry>
-	<mesh filename="package://wally_description/meshes/RODA_A.dae" />
+	<mesh filename="package://wally_description/meshes/RODA.dae" />
       </geometry>
     </collision>
